File: hardware/linux-based-scout-uav/gnss.kicad_sch (KiCad schematic)
At the start: 1 part, among them U4 LC76G

Commit message: Schematic update
Connections:
- net GND: now reaches U4.1 (GND), U4.10 (GND), U4.12 (GND), U4.28 (GND)
Changed lines of the file:
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@@
 	(generator_version "8.0")
 	(paper "A3")
+	(wire
+		(pts
+			(xy 224.79 148.59) (xy 234.95 148.59)
+		)
+		(stroke
+			(width 0)
+			(type default)
+		)
+	)
+	(wire
+		(pts
+			(xy 234.95 148.59) (xy 234.95 158.75)
+		)
+		(stroke
+			(width 0)
+			(type default)
+		)
+	)
 	(symbol
 		(lib_id "LC76G:LC76G")
@@
 					(unit 1)
 				)
+			)
+		)
+	)
+	(symbol
+		(lib_id "power:GND")
+		(at 234.95 158.75 0)
+		(unit 1)
+		(exclude_from_sim no)
+		(in_bom yes)
+		(on_board yes)
+		(dnp no)
+		(fields_autoplaced yes)
+		(property "Reference" "#PWR016"
+			(at 234.95 165.1 0)
+			(effects
+				(font
+					(size 1.27 1.27)
+				)
+				(hide yes)
+			)
+		)
+		(property "Value" "GND"
+			(at 234.95 163.83 0)
+			(effects
+				(font
+					(size 1.27 1.27)
+				)
+			)
+		)
+		(property "Footprint" ""
+			(at 234.95 158.75 0)
+			(effects
+				(font
+					(size 1.27 1.27)
+				)
+				(hide yes)
+			)
+		)
+		(property "Datasheet" ""
+			(at 234.95 158.75 0)
+			(effects
+				(font
+					(size 1.27 1.27)
+				)
+				(hide yes)
+			)
+		)
+		(property "Description" "Power symbol creates a global label with name \"GND\" , ground"
+			(at 234.95 158.75 0)
+			(effects
+				(font
+					(size 1.27 1.27)
+				)
+				(hide yes)
+			)
+		)
+		(pin "1"
+		)
+		(instances
+			(project ""
+				(path "/e9b29a7c-bbe5-4ab4-acee-985586e1266a/e37a2e8f-5c01-4343-930e-9e20e12f83a8"
+					(reference "#PWR016")
+					(unit 1)
+				)

Commit message: Schematic update
Other:
- note added: "GNSS"
Changed lines of the file:
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@@
+		)
+	)
+	(text "GNSS"
+		(exclude_from_sim no)
+		(at 203.962 27.178 0)
+		(effects
+			(font
+				(face "KiCad Font")
+				(size 10.16 10.16)
+			)
 		)
 	)
