File: hardware/linux-based-scout-uav/osd32mp1-1-power.kicad_sch (KiCad schematic)
At the start: 4 parts, among them SW1 SW_DIP_x04, U1 OSD32MP157C-512M-IAA

Commit message: Schematic/board update
Parts:
- added TP10, TP11, TP12, TP13, TP14, TP15, TP16, TP17, TP18, TP3, TP4, TP5, TP6, TP7, TP8, TP9: TestPoint, symbol Connector:TestPoint
Connections:
- net at U1.D5 (PWR_ON/PMIC_PWRCTRL): now also TP14.1
- net at U1.D6 (PC13/PMIC_WAKEUP): now also TP13.1
- net at U1.J12 (VTT_DDR): now also TP5.1
- net at U1.J2 (HSE_OSC_TP): now also TP11.1
- net at U1.K12 (VDD_DDR): now also TP4.1
- net at U1.K6 (PWR_LP): now also TP15.1
- net at U1.L12 (VREF_DDR): now also TP6.1
- net at U1.L3 (PA0/PMIC_INTN): now also TP12.1
- net at U1.L6 (PDR_ON_CORE): now also TP17.1
- net at U1.M6 (PDR_ON): now also TP16.1
- net at U1.N4 (NRST_CORE): now also TP18.1
- net at U1.R4 (VDD_CORE): now also TP3.1
- net at U1.R5 (VDD3V3_USB): now also TP7.1
- net at U1.R6 (VDD1V2_DSI_REG): now also TP10.1
- net at U1.R7 (VDDA1V8_REG): now also TP9.1
- net at U1.R8 (VDDA1V1_REG): now also TP8.1
