File: hardware/linux-based-scout-uav/osd32mp1-2.kicad_sch (KiCad schematic)
At the start: 7 parts, among them J3 TC2050-IDC-NL, U1 OSD32MP157C-512M-IAA, Y1 ABS05-32.768KHZ-7-T

Commit message: schematic update
schematic update
Parts:
- added TP1, TP2: TestPoint, symbol Connector:TestPoint
Connections:
- net at U1.L1 (ANA0): now also TP1.1
- net at U1.L2 (ANA1): now also TP2.1
Changed lines of the file:
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@@
+	(wire
+		(pts
+			(xy 110.49 135.89) (xy 115.57 135.89)
+		)
+		(stroke
+			(width 0)
+			(type default)
+		)
+	)
+	(wire
+		(pts
+			(xy 128.27 138.43) (xy 128.27 132.08)
+		)
+		(stroke
+			(width 0)
+			(type default)
+		)
+	)
 	(wire
 		(pts
@@
 	(wire
 		(pts
+			(xy 110.49 138.43) (xy 128.27 138.43)
+		)
+		(stroke
+			(width 0)
+			(type default)
+		)
+	)
+	(wire
+		(pts
 			(xy 40.64 231.14) (xy 68.58 231.14)
 		)
@@
 		(pts
 			(xy 294.64 128.27) (xy 294.64 138.43)
+		)
+		(stroke
+			(width 0)
+			(type default)
+		)
+	)
+	(wire
+		(pts
+			(xy 115.57 135.89) (xy 115.57 132.08)
 		)
 		(stroke
@@
 				(justify right)
 				(hide yes)
+			)
+		)
+	)
+	(symbol
+		(lib_id "Connector:TestPoint")
+		(at 128.27 132.08 0)
+		(unit 1)
+		(exclude_from_sim no)
+		(in_bom yes)
+		(on_board yes)
+		(dnp no)
+		(fields_autoplaced yes)
+		(property "Reference" "TP2"
+			(at 130.81 127.5079 0)
+			(effects
+				(font
+					(size 1.27 1.27)
+				)
+				(justify left)
+			)
+		)
+		(property "Value" "TestPoint"
+			(at 130.81 130.0479 0)
+			(effects
+				(font
+					(size 1.27 1.27)
+				)
+				(justify left)
+			)
+		)
+		(property "Footprint" ""
+			(at 133.35 132.08 0)
+			(effects
+				(font
+					(size 1.27 1.27)
+				)
+				(hide yes)
+			)
+		)
+		(property "Datasheet" "~"
+			(at 133.35 132.08 0)
+			(effects
+				(font
+					(size 1.27 1.27)
+				)
+				(hide yes)
+			)
+		)
+		(property "Description" "test point"
+			(at 128.27 132.08 0)
+			(effects
+				(font
+					(size 1.27 1.27)
+				)
+				(hide yes)
+			)
+		)
+		(pin "1"
+		)
+		(instances
+			(project ""
+				(path "/e9b29a7c-bbe5-4ab4-acee-985586e1266a/ec3f42cd-4cf8-4535-a092-0d9cee8969c9"
+					(reference "TP2")
+					(unit 1)
+				)
 			)
 		)
@@
 				)
 			)
+		)
+	)
+	(symbol
+		(lib_id "Connector:TestPoint")
+		(at 115.57 132.08 0)
+		(unit 1)
+		(exclude_from_sim no)
+		(in_bom yes)
+		(on_board yes)
+		(dnp no)
+		(fields_autoplaced yes)
+		(property "Reference" "TP1"
+			(at 118.11 127.5079 0)
+			(effects
+				(font
+					(size 1.27 1.27)
+				)
+				(justify left)
+			)
+		)
+		(property "Value" "TestPoint"
+			(at 118.11 130.0479 0)
+			(effects
+				(font
+					(size 1.27 1.27)
+				)
+				(justify left)
+			)
+		)
+		(property "Footprint" ""
+			(at 120.65 132.08 0)
+			(effects
+				(font
+					(size 1.27 1.27)
+				)
+				(hide yes)
+			)
+		)
+		(property "Datasheet" "~"
+			(at 120.65 132.08 0)
+			(effects
+				(font
+					(size 1.27 1.27)
+				)
+				(hide yes)
+			)
+		)
+		(property "Description" "test point"
+			(at 115.57 132.08 0)
+			(effects
+				(font
+					(size 1.27 1.27)
+				)
+				(hide yes)
+			)
+		)
+		(pin "1"
+		)
+		(instances
+			(project ""
+				(path "/e9b29a7c-bbe5-4ab4-acee-985586e1266a/ec3f42cd-4cf8-4535-a092-0d9cee8969c9"
+					(reference "TP1")
+					(unit 1)
+				)
+			)

Commit message: Schematic/board update
Connections:
- net MMC2_D7: now reaches U1.R16 (PC7)
- net MMC2_D0: now reaches U1.T14 (PB14)
- net MMC2_D4: now reaches U1.T17 (PA8)
- net MMC2_D5: now reaches U1.U12 (PA9)
- net MMC2_D3: now reaches U1.U14 (PB4)
- net MMC2_D1: now reaches U1.V13 (PB15)
- net MMC2_D2: now reaches U1.V14 (PB3)
Other:
- note added: "MMC2_D[0..7] Bus"

Commit message: Schematic and board update
Connections:
- net USB_DM1 renamed USB_DN
- net USB_DM2 renamed USB_2_DN
- net USB_DP1 renamed USB_DP
- net USB_DP2 renamed USB_2_DP
Changed lines of the file:
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@@
 		)
 	)
-	(global_label "USB_DP2"
+	(global_label "USB_2_DP"
 		(shape bidirectional)
 		(at 38.1 163.83 180)
@@
 		)
 		(property "Intersheetrefs" "${INTERSHEET_REFS}"
-			(at 25.4764 163.83 0)
-			(effects
-				(font
-					(size 1.27 1.27)
-				)
-				(justify right)
-				(hide yes)
-			)
-		)
-	)
-	(global_label "USB_DM2"
+			(at 24.5088 163.83 0)
+			(effects
+				(font
+					(size 1.27 1.27)
+				)
+				(justify right)
+				(hide yes)
+			)
+		)
+	)
+	(global_label "USB_2_DN"
 		(shape bidirectional)
 		(at 38.1 161.29 180)
@@
 		)
 		(property "Intersheetrefs" "${INTERSHEET_REFS}"
-			(at 25.295 161.29 0)
+			(at 24.4483 161.29 0)
 			(effects
 				(font
@@
 		)
 	)
-	(global_label "USB_DM1"
+	(global_label "USB_DN"
 		(shape bidirectional)
 		(at 38.1 151.13 180)
@@
 		)
 		(property "Intersheetrefs" "${INTERSHEET_REFS}"
-			(at 25.295 151.13 0)
+			(at 26.6254 151.13 0)
 			(effects
 				(font
@@
 		)
 	)
-	(global_label "USB_DP1"
+	(global_label "USB_DP"
 		(shape bidirectional)
 		(at 38.1 153.67 180)
@@
 		)
 		(property "Intersheetrefs" "${INTERSHEET_REFS}"
-			(at 25.4764 153.67 0)
-			(effects
-				(font
+			(at 26.6859 153.67 0)
+			(effects
+				(font
