File: hardware/linux-based-scout-uav/quectel-m65-1.kicad_sch (KiCad schematic)
At the start: 1 part, among them U3 M65

Commit message: Schematic update
Connections:
- net GND: now reaches U3.1 (AGND)
- net GND: now also U3.10 (SIM_GND), U3.27 (GND), U3.34 (GND), U3.36 (GND), U3.37 (GND), U3.40 (GND), U3.41 (GND)
Changed lines of the file:
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@@
 	(generator_version "8.0")
 	(paper "A3")
+	(junction
+		(at 259.08 149.86)
+		(diameter 0)
+		(color 0 0 0 0)
+	)
+	(junction
+		(at 259.08 152.4)
+		(diameter 0)
+		(color 0 0 0 0)
+	)
+	(wire
+		(pts
+			(xy 248.92 147.32) (xy 259.08 147.32)
+		)
+		(stroke
+			(width 0)
+			(type default)
+		)
+	)
+	(wire
+		(pts
+			(xy 248.92 149.86) (xy 259.08 149.86)
+		)
+		(stroke
+			(width 0)
+			(type default)
+		)
+	)
+	(wire
+		(pts
+			(xy 259.08 152.4) (xy 259.08 162.56)
+		)
+		(stroke
+			(width 0)
+			(type default)
+		)
+	)
+	(wire
+		(pts
+			(xy 248.92 152.4) (xy 259.08 152.4)
+		)
+		(stroke
+			(width 0)
+			(type default)
+		)
+	)
+	(wire
+		(pts
+			(xy 259.08 149.86) (xy 259.08 152.4)
+		)
+		(stroke
+			(width 0)
+			(type default)
+		)
+	)
+	(wire
+		(pts
+			(xy 259.08 147.32) (xy 259.08 149.86)
+		)
+		(stroke
+			(width 0)
+			(type default)
+		)
+	)
 	(symbol
 		(lib_id "M65:M65")
@@
 					(unit 1)
 				)
+			)
+		)
+	)
+	(symbol
+		(lib_id "power:GND")
+		(at 259.08 162.56 0)
+		(unit 1)
+		(exclude_from_sim no)
+		(in_bom yes)
+		(on_board yes)
+		(dnp no)
+		(fields_autoplaced yes)
+		(property "Reference" "#PWR015"
+			(at 259.08 168.91 0)
+			(effects
+				(font
+					(size 1.27 1.27)
+				)
+				(hide yes)
+			)
+		)
+		(property "Value" "GND"
+			(at 259.08 167.64 0)
+			(effects
+				(font
+					(size 1.27 1.27)
+				)
+			)
+		)
+		(property "Footprint" ""
+			(at 259.08 162.56 0)
+			(effects
+				(font
+					(size 1.27 1.27)
+				)
+				(hide yes)
+			)
+		)
+		(property "Datasheet" ""
+			(at 259.08 162.56 0)
+			(effects
+				(font
+					(size 1.27 1.27)
+				)
+				(hide yes)
+			)
+		)
+		(property "Description" "Power symbol creates a global label with name \"GND\" , ground"
+			(at 259.08 162.56 0)
+			(effects
+				(font
+					(size 1.27 1.27)
+				)
+				(hide yes)
+			)
+		)
+		(pin "1"
+		)
+		(instances
+			(project ""
+				(path "/e9b29a7c-bbe5-4ab4-acee-985586e1266a/b0fb3ce5-1b3a-433c-9ac4-077516adadc9"
+					(reference "#PWR015")
+					(unit 1)
+				)

Commit message: Schematic update
Parts:
- added C3: 100nF, Capacitor_SMD:C_0402_1005Metric, symbol Device:C
- added J4: 0786463001, 0786463001:MOLEX_0786463001, symbol 0786463001:0786463001
- added R13, R14, R15: 22R, Resistor_SMD:R_0402_1005Metric, symbol Device:R
Connections:
- net GND: now also C3.2, J4.C5 (GND), J4.G1 (GND), J4.G2 (GND), J4.G3 (GND), J4.G4 (GND), J4.G5 (GND), J4.G6 (GND)
- net at U3.11 (SIM_DATA): now also R13.2
- net at U3.12 (SIM_RST): now also R15.2
- net at U3.13 (SIM_CLK): now also R14.2
- net SIM_VDD: now reaches U3.14 (SIM_VDD)
- net SIM_VDD: now also C3.1, J4.C1 (VCC)
- new net SIM_CLK: J4.C3 (CLK), R14.1
- new net SIM_DATA: J4.C7 (I/O), R13.1
- new net SIM_RST: J4.C2 (RST), R15.1
Other:
- note added: "GSM/GPRS 2G Comms"
- note added: "Micro SIM card socket"
